File: ClockController.X/Hardware/Clock_Controller_6.kicad_sch (KiCad schematic)
At the start: 7 parts

Commit message: Cleaned up a bunch of labels
Changed lines of the file:
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@@
-	(wire
-		(pts
-			(xy 111.76 78.74) (xy 111.76 72.39)
-		)
-		(stroke
-			(width 0.25)
-			(type solid)
-		)
-	)
 	(wire
 		(pts
@@
 		)
 	)
+	(wire
+		(pts
+			(xy 111.76 72.39) (xy 111.76 78.74)
+		)
+		(stroke
+			(width 0)
+			(type default)
+		)
+	)
 	(text "10k"
 		(exclude_from_sim no)
@@
 	(text "RC5"
 		(exclude_from_sim no)
-		(at 122.396 65.538 90)
-		(effects
-			(font
-				(size 1.48 1.48)
-			)
-			(justify left bottom)
+		(at 125.222 61.722 0)
+		(effects
+			(font
+				(size 1.48 1.48)
+			)
+			(justify right bottom)
 		)
 	)
 	(text "RC3"
 		(exclude_from_sim no)
-		(at 173.196 134.118 90)
+		(at 171.958 136.144 0)
 		(effects
 			(font
@@
 	(text "RC4"
 		(exclude_from_sim no)
-		(at 122.396 134.154 90)
-		(effects
-			(font
-				(size 1.48 1.48)
-			)
-			(justify left bottom)
+		(at 125.476 136.144 0)
+		(effects
+			(font
+				(size 1.48 1.48)
+			)
+			(justify right bottom)
 		)
 	)
@@
 	(global_label "Rotary_A"
 		(shape bidirectional)
-		(at 111.76 78.74 0)
+		(at 111.76 72.39 180)
 		(fields_autoplaced yes)
 		(effects
@@
 				(size 1.016 1.016)
 			)
-			(justify left)
+			(justify right)
 		)
 		(property "Intersheetrefs" "${INTERSHEET_REFS}"
-			(at 121.52 78.74 0)
+			(at 102 72.39 0)
 			(effects
 				(font
 					(size 1.27 1.27)
 				)
-				(justify left)
+				(justify right)
 				(hide yes)
 			)
