File: ClockController.X/Hardware/USB PD.kicad_sch (KiCad schematic)
At the start: 13 parts, among them J1 UJC-VP-3-SMT-TR, Q1 DMG7430LFG-7, U4 AP33772DKZ-13

Commit message: Converting to single board layout
Connections:
- net 3.3V: now reaches U4.12 (V3VD)
- net 3.3V: now also UNK5V0.2 (A)
- net 5V LED Limit renamed 3V LED Limit
- net V5V renamed 5V
- net 5V: no longer UNK5V0.2 (A)
- no-connect marks 12 -> 11
Changed lines of the file:
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@@
 	(generator "eeschema")
 	(generator_version "9.0")
-	(paper "A4")
+	(paper "USLetter")
 	(junction
 		(at 69.85 118.11)
@@
 	)
 	(junction
-		(at 53.34 137.16)
-		(diameter 0)
-		(color 0 0 0 0)
-	)
-	(junction
 		(at 83.82 66.04)
 		(diameter 0)
@@
 	)
 	(no_connect
-		(at 212.09 69.85)
-	)
-	(no_connect
 		(at 166.37 87.63)
 	)
@@
 	(wire
 		(pts
-			(xy 53.34 137.16) (xy 53.34 142.24)
+			(xy 219.71 69.85) (xy 212.09 69.85)
 		)
 		(stroke
@@
 		(pts
 			(xy 212.09 97.79) (xy 215.9 97.79)
-		)
-		(stroke
-			(width 0)
-			(type default)
-		)
-	)
-	(wire
-		(pts
-			(xy 53.34 137.16) (xy 49.53 137.16)
 		)
 		(stroke
@@
 	(wire
 		(pts
-			(xy 53.34 137.16) (xy 59.69 137.16)
-		)
-		(stroke
-			(width 0)
-			(type default)
-		)
-	)
-	(wire
-		(pts
 			(xy 157.48 72.39) (xy 166.37 72.39)
 		)
@@
 		(pts
 			(xy 69.85 110.49) (xy 69.85 115.57)
+		)
+		(stroke
+			(width 0)
+			(type default)
+		)
+	)
+	(wire
+		(pts
+			(xy 57.15 137.16) (xy 59.69 137.16)
 		)
 		(stroke
@@
 		)
 	)
+	(label "3.3V"
+		(at 215.9 69.85 180)
+		(effects
+			(font
+				(size 1.27 1.27)
+			)
+			(justify right bottom)
+		)
+	)
 	(label "VBUS Enable"
 		(at 120.65 78.74 0)
@@
 		)
 	)
+	(label "3.3V"
+		(at 57.15 137.16 180)
+		(effects
+			(font
+				(size 1.27 1.27)
+			)
+			(justify right)
+		)
+	)
 	(label "IFB"
 		(at 160.02 72.39 0)
@@
 		)
 	)
-	(label "5V LED Limit"
+	(label "3V LED Limit"
 		(at 72.39 137.16 270)
 		(effects
@@
 			)
 			(justify left bottom)
-		)
-	)
-	(global_label "V5V"
-		(shape bidirectional)
-		(at 166.37 85.09 180)
-		(fields_autoplaced yes)
-		(effects
-			(font
-				(size 1.016 1.016)
-			)
-			(justify right)
-		)
-		(property "Intersheetrefs" "${INTERSHEET_REFS}"
-			(at 160.3837 85.09 0)
-			(effects
-				(font
-					(size 1.27 1.27)
-				)
-				(justify right)
-				(hide yes)
-			)
 		)
 	)
@@
 		)
 	)
-	(global_label "V5V"
-		(shape bidirectional)
-		(at 53.34 142.24 270)
-		(fields_autoplaced yes)
-		(effects
-			(font
-				(size 1.016 1.016)
-			)
-			(justify right)
-		)
-		(property "Intersheetrefs" "${INTERSHEET_REFS}"
-			(at 53.34 148.2263 90)
-			(effects
-				(font
-					(size 1.27 1.27)
-				)
-				(justify right)
-				(hide yes)
-			)
-		)
-	)
 	(hierarchical_label "SDA"
 		(shape bidirectional)
@@
 		)
 	)
+	(hierarchical_label "3.3V"
+		(shape bidirectional)
+		(at 219.71 69.85 0)
+		(effects
+			(font
+				(size 1.27 1.27)
+			)
+			(justify left)
+		)
+	)
 	(hierarchical_label "5V"
 		(shape output)
-		(at 49.53 137.16 180)
+		(at 166.37 85.09 180)
 		(effects
 			(font
@@
 		)
 	)
+	(netclass_flag ""
+		(length 2.54)
+		(shape round)
+		(at 67.31 92.71 0)
+		(fields_autoplaced yes)
+		(effects
+			(font
+				(size 1.27 1.27)
+			)
+			(justify left bottom)
+		)
+		(property "Netclass" "Extra Thicc"
+			(at 68.0085 90.17 0)
+			(effects
+				(font
+					(size 1.27 1.27)
+				)
+				(justify left)
+			)
+		)
+		(property "Component Class" ""
+			(at -144.78 24.13 0)
+			(effects
+				(font
+					(size 1.27 1.27)
+					(italic yes)
+				)
+			)
+		)
+	)
+	(netclass_flag ""
+		(length 2.54)
+		(shape round)
+		(at 147.32 72.39 0)
+		(effects
+			(font
+				(size 1.27 1.27)
+			)
+			(justify left bottom)
+		)
+		(property "Netclass" "Thicc"
+			(at 147.32 68.58 90)
+			(effects
+				(font
+					(size 1.27 1.27)
+				)
+				(justify left)
+			)
+		)
+		(property "Component Class" ""
+			(at -106.68 12.7 0)
+			(effects
+				(font
+					(size 1.27 1.27)
+					(italic yes)
+				)
+			)
+		)
+	)
+	(netclass_flag ""
+		(length 2.54)
+		(shape round)
+		(at 217.17 69.85 0)
+		(effects
+			(font
+				(size 1.27 1.27)
+			)
+			(justify left bottom)
+		)
+		(property "Netclass" "Thicc"
+			(at 217.17 66.04 90)
+			(effects
+				(font
+					(size 1.27 1.27)
+				)
+				(justify left)
+			)
+		)
+		(property "Component Class" ""
+			(at 0 10.16 0)
+			(effects
+				(font
+					(size 1.27 1.27)
+					(italic yes)
+				)
+			)
+		)
+	)
