File: ClockController.X/Hardware/USB PD.kicad_sch (KiCad schematic)
At the start: 14 parts, among them J1 UJC-VP-3-SMT-TR, Q1 DMG7430LFG-7, U4 AP33772DKZ-13

Commit message: Updated most footprints
Parts:
- C1: footprint Clock Controller:CAP_0805 -> Capacitor_SMD:C_0805_2012Metric
- C4: footprint Clock Controller:CAP_1206 -> Capacitor_SMD:C_1206_3216Metric
- J1: footprint CUI_UJC-VP-3-SMT-TR -> Connector USB:CUI_UJC-VP-3-SMT-TR
- PD0: footprint Clock Controller:LED_1206(3216_METRIC)_N_BLUE -> LED_SMD:LED_1206_3216Metric
- Q1: footprint Clock Controller:POWERDI3333-8 -> Diodes Incorporated:TRANS_DMP3017SFGQ-7
- R10, R11, R5, R6, R9: footprint Clock Controller:RES_0805 -> Resistor_SMD:R_0805_2012Metric
- R7: footprint Clock Controller:RES_1206 -> Resistor_SMD:R_1206_3216Metric
- U4: footprint Clock Controller:W-QFN4040-24_(TYPE_A1) -> Package_DFN_QFN:QFN-24-1EP_4x4mm_P0.5mm_EP2.7x2.7mm
- UNK5V0: footprint Clock Controller:LED_1206(3216_METRIC)_N_GREEN -> LED_SMD:LED_1206_3216Metric
Changed lines of the file:
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@@
 	(wire
 		(pts
-			(xy 149.86 72.39) (xy 142.24 72.39)
-		)
-		(stroke
-			(width 0.25)
-			(type solid)
-		)
-	)
-	(wire
-		(pts
-			(xy 212.09 85.09) (xy 234.95 85.09)
-		)
-		(stroke
-			(width 0.25)
-			(type solid)
-		)
-	)
-	(wire
-		(pts
-			(xy 64.77 92.71) (xy 69.85 92.71)
-		)
-		(stroke
-			(width 0.25)
-			(type solid)
-		)
-	)
-	(wire
-		(pts
-			(xy 87.63 73.66) (xy 99.06 73.66)
-		)
-		(stroke
-			(width 0.25)
-			(type solid)
-		)
-	)
-	(wire
-		(pts
-			(xy 64.77 102.87) (xy 78.74 102.87)
-		)
-		(stroke
-			(width 0.25)
-			(type solid)
-		)
-	)
-	(wire
-		(pts
-			(xy 123.19 120.65) (xy 133.35 120.65)
-		)
-		(stroke
-			(width 0.25)
-			(type solid)
-		)
-	)
-	(wire
-		(pts
-			(xy 78.74 102.87) (xy 78.74 106.68)
-		)
-		(stroke
-			(width 0.25)
-			(type solid)
-		)
-	)
-	(wire
-		(pts
-			(xy 234.95 130.81) (xy 234.95 140.716)
-		)
-		(stroke
-			(width 0.25)
-			(type solid)
-		)
-	)
-	(wire
-		(pts
-			(xy 69.85 115.57) (xy 69.85 113.03)
+			(xy 142.24 72.39) (xy 149.86 72.39)
 		)
 		(stroke
@@
 	(wire
 		(pts
-			(xy 133.35 90.17) (xy 166.37 90.17)
-		)
-		(stroke
-			(width 0.25)
-			(type solid)
-		)
-	)
-	(wire
-		(pts
-			(xy 160.02 97.79) (xy 166.37 97.79)
-		)
-		(stroke
-			(width 0.25)
-			(type solid)
-		)
-	)
-	(wire
-		(pts
-			(xy 80.01 73.66) (xy 76.2 73.66)
-		)
-		(stroke
-			(width 0.25)
-			(type solid)
-		)
-	)
-	(wire
-		(pts
-			(xy 88.9 100.33) (xy 88.9 106.68)
-		)
-		(stroke
-			(width 0.25)
-			(type solid)
-		)
-	)
-	(wire
-		(pts
-			(xy 69.85 107.95) (xy 69.85 110.49)
-		)
-		(stroke
-			(width 0.25)
-			(type solid)
-		)
-	)
-	(wire
-		(pts
-			(xy 69.85 110.49) (xy 69.85 107.95)
+			(xy 212.09 85.09) (xy 234.95 85.09)
+		)
+		(stroke
+			(width 0.25)
+			(type solid)
+		)
+	)
+	(wire
+		(pts
+			(xy 64.77 92.71) (xy 69.85 92.71)
+		)
+		(stroke
+			(width 0.25)
+			(type solid)
+		)
+	)
+	(wire
+		(pts
+			(xy 87.63 73.66) (xy 99.06 73.66)
+		)
+		(stroke
+			(width 0.25)
+			(type solid)
+		)
+	)
+	(wire
+		(pts
+			(xy 64.77 102.87) (xy 78.74 102.87)
+		)
+		(stroke
+			(width 0.25)
+			(type solid)
+		)
+	)
+	(wire
+		(pts
+			(xy 123.19 120.65) (xy 133.35 120.65)
+		)
+		(stroke
+			(width 0.25)
+			(type solid)
+		)
+	)
+	(wire
+		(pts
+			(xy 78.74 102.87) (xy 78.74 106.68)
+		)
+		(stroke
+			(width 0.25)
+			(type solid)
+		)
+	)
+	(wire
+		(pts
+			(xy 234.95 130.81) (xy 234.95 140.716)
+		)
+		(stroke
+			(width 0.25)
+			(type solid)
+		)
+	)
+	(wire
+		(pts
+			(xy 69.85 115.57) (xy 69.85 113.03)
 		)
 		(stroke
@@
 	(wire
 		(pts
-			(xy 64.77 100.33) (xy 88.9 100.33)
-		)
-		(stroke
-			(width 0.25)
-			(type solid)
-		)
-	)
-	(wire
-		(pts
-			(xy 129.54 82.55) (xy 123.19 82.55)
-		)
-		(stroke
-			(width 0.25)
-			(type solid)
-		)
-	)
-	(wire
-		(pts
-			(xy 157.48 72.39) (xy 166.37 72.39)
-		)
-		(stroke
-			(width 0.25)
-			(type solid)
-		)
-	)
-	(wire
-		(pts
-			(xy 88.9 123.19) (xy 88.9 119.38)
+			(xy 133.35 90.17) (xy 166.37 90.17)
+		)
+		(stroke
+			(width 0.25)
+			(type solid)
+		)
+	)
+	(wire
+		(pts
+			(xy 160.02 97.79) (xy 166.37 97.79)
+		)
+		(stroke
+			(width 0.25)
+			(type solid)
+		)
+	)
+	(wire
+		(pts
+			(xy 80.01 73.66) (xy 76.2 73.66)
+		)
+		(stroke
+			(width 0.25)
+			(type solid)
+		)
+	)
+	(wire
+		(pts
+			(xy 88.9 100.33) (xy 88.9 106.68)
+		)
+		(stroke
+			(width 0.25)
+			(type solid)
+		)
+	)
+	(wire
+		(pts
+			(xy 69.85 107.95) (xy 69.85 110.49)
+		)
+		(stroke
+			(width 0.25)
+			(type solid)
+		)
+	)
+	(wire
+		(pts
+			(xy 69.85 110.49) (xy 69.85 107.95)
 		)
 		(stroke
@@
 	(wire
 		(pts
-			(xy 214.63 105.41) (xy 99.06 105.41)
-		)
-		(stroke
-			(width 0.25)
-			(type solid)
-		)
-	)
-	(wire
-		(pts
-			(xy 99.06 105.41) (xy 99.06 95.25)
-		)
-		(stroke
-			(width 0.25)
-			(type solid)
-		)
-	)
-	(wire
-		(pts
-			(xy 106.68 120.65) (xy 110.49 120.65)
+			(xy 64.77 100.33) (xy 88.9 100.33)
+		)
+		(stroke
+			(width 0.25)
+			(type solid)
+		)
+	)
+	(wire
+		(pts
+			(xy 129.54 82.55) (xy 123.19 82.55)
+		)
+		(stroke
+			(width 0.25)
+			(type solid)
+		)
+	)
+	(wire
+		(pts
+			(xy 88.9 123.19) (xy 88.9 119.38)
 		)
 		(stroke
@@
 	(wire
 		(pts
+			(xy 214.63 105.41) (xy 99.06 105.41)
+		)
+		(stroke
+			(width 0.25)
+			(type solid)
+		)
+	)
+	(wire
+		(pts
+			(xy 99.06 105.41) (xy 99.06 95.25)
+		)
+		(stroke
+			(width 0.25)
+			(type solid)
+		)
+	)
+	(wire
+		(pts
+			(xy 106.68 120.65) (xy 110.49 120.65)
+		)
+		(stroke
+			(width 0)
+			(type default)
+		)
+	)
+	(wire
+		(pts
 			(xy 64.77 115.57) (xy 69.85 115.57)
+		)
+		(stroke
+			(width 0)
+			(type default)
+		)
+	)
+	(wire
+		(pts
+			(xy 157.48 72.39) (xy 166.37 72.39)
 		)
 		(stroke
@@
 			)
 		)
-		(property "Footprint" "Clock Controller:CAP_1206"
+		(property "Footprint" "Capacitor_SMD:C_1206_3216Metric"
 			(at 83.82 73.66 0)
 			(effects
@@
 			)
 		)
-		(property "Footprint" "Clock Controller:LED_1206(3216_METRIC)_N_BLUE"
+		(property "Footprint" "LED_SMD:LED_1206_3216Metric"
 			(at 234.95 101.6 0)
 			(effects
@@
 			)
 		)
-		(property "Footprint" "Clock Controller:RES_1206"
+		(property "Footprint" "Resistor_SMD:R_1206_3216Metric"
 			(at 116.84 95.25 0)
 			(effects
@@
 			)
 		)
-		(property "Footprint" "Clock Controller:RES_0805"
+		(property "Footprint" "Resistor_SMD:R_0805_2012Metric"
 			(at 116.84 82.55 0)
 			(effects
@@
 			)
 		)
-		(property "Footprint" "Clock Controller:CAP_0805"
+		(property "Footprint" "Capacitor_SMD:C_0805_2012Metric"
 			(at 153.67 72.39 0)
 			(effects
@@
 			)
 		)
-		(property "Footprint" "CUI_UJC-VP-3-SMT-TR"
+		(property "Footprint" "Connector USB:CUI_UJC-VP-3-SMT-TR"
 			(at 52.07 100.33 0)
 			(effects
@@
 			)
 		)
-		(property "Footprint" "Clock Controller:RES_0805"
+		(property "Footprint" "Resistor_SMD:R_0805_2012Metric"
 			(at 139.7 120.65 0)
 			(effects
@@
 			)
 		)
-		(property "Footprint" "Clock Controller:RES_0805"
+		(property "Footprint" "Resistor_SMD:R_0805_2012Metric"
 			(at 234.95 124.46 0)
 			(effects
@@
 			)
 		)
-		(property "Footprint" "Clock Controller:LED_1206(3216_METRIC)_N_GREEN"
+		(property "Footprint" "LED_SMD:LED_1206_3216Metric"
 			(at 116.84 120.65 0)
 			(effects
@@
 			)
 		)
-		(property "Footprint" "Clock Controller:RES_0805"
+		(property "Footprint" "Resistor_SMD:R_0805_2012Metric"
 			(at 88.9 113.03 0)
 			(effects
@@
 			)
 		)
-		(property "Footprint" "Clock Controller:W-QFN4040-24_(TYPE_A1)"
+		(property "Footprint" "Package_DFN_QFN:QFN-24-1EP_4x4mm_P0.5mm_EP2.7x2.7mm"
 			(at 212.09 97.79 0)
 			(effects
@@
 			)
 		)
-		(property "Footprint" "Clock Controller:POWERDI3333-8"
+		(property "Footprint" "Diodes Incorporated:TRANS_DMP3017SFGQ-7"
 			(at 107.95 82.55 0)
 			(effects
@@
 			)
 		)
-		(property "Footprint" "Clock Controller:RES_0805"
+		(property "Footprint" "Resistor_SMD:R_0805_2012Metric"
 			(at 78.74 113.03 0)
 			(effects

Commit message: Fixed footprint issue with Q1
Parts:
- Q1: footprint Diodes Incorporated:TRANS_DMP3017SFGQ-7 -> Diodes Incorporated:PowerDI3333-8
Changed lines of the file:
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@@
+	(wire
+		(pts
+			(xy 166.37 92.71) (xy 129.54 92.71)
+		)
+		(stroke
+			(width 0.25)
+			(type solid)
+		)
+	)
+	(wire
+		(pts
+			(xy 234.95 107.95) (xy 234.95 118.11)
+		)
+		(stroke
+			(width 0.25)
+			(type solid)
+		)
+	)
+	(wire
+		(pts
+			(xy 133.35 73.66) (xy 133.35 90.17)
+		)
+		(stroke
+			(width 0.25)
+			(type solid)
+		)
+	)
 	(wire
 		(pts
@@
 		)
 		(stroke
-			(width 0.25)
-			(type solid)
-		)
-	)
-	(wire
-		(pts
-			(xy 166.37 92.71) (xy 129.54 92.71)
-		)
-		(stroke
-			(width 0.25)
-			(type solid)
-		)
-	)
-	(wire
-		(pts
-			(xy 234.95 107.95) (xy 234.95 118.11)
-		)
-		(stroke
-			(width 0.25)
-			(type solid)
-		)
-	)
-	(wire
-		(pts
-			(xy 133.35 73.66) (xy 133.35 90.17)
-		)
-		(stroke
-			(width 0.25)
-			(type solid)
+			(width 0)
+			(type default)
 		)
 	)
@@
 			)
 		)
-		(property "Footprint" "Diodes Incorporated:TRANS_DMP3017SFGQ-7"
+		(property "Footprint" "Diodes Incorporated:PowerDI3333-8"
 			(at 107.95 82.55 0)
 			(effects

Commit message: Unsaved changes
Parts:
- Q1: symbol Clock Controller-eagle-import:DMG7430LFG-7 -> Transistor_FET_:DMG7430LFG-7
Connections:
- net +20V: now also Q1.3 (S)
- net VBUS: now also Q1.6 (D), Q1.7 (D), Q1.8 (D)
Changed lines of the file:
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@@
 	)
 	(symbol
-		(lib_id "Clock Controller-eagle-import:DMG7430LFG-7")
+		(lib_id "Transistor_FET_:DMG7430LFG-7")
 		(at 107.95 82.55 180)
 		(unit 1)
@@
 		)
 		(property "Footprint" "Diodes Incorporated:PowerDI3333-8"
-			(at 107.95 82.55 0)
+			(at 100.33 96.774 0)
 			(effects
 				(font
@@
 		(pin "2"
 		)
+		(pin "6"
+		)
+		(pin "8"
+		)
+		(pin "3"
+		)
+		(pin "7"
+		)
 		(instances

Commit message: Replacing many thin traces with poured zones.
Changed lines of the file:
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@@
 (kicad_sch
-	(version 20231120)
+	(version 20250114)
 	(generator "eeschema")
-	(generator_version "8.0")
+	(generator_version "9.0")
 	(paper "A4")
+	(text "0.01"
+		(exclude_from_sim no)
+		(at 114.857 93.98 0)
+		(effects
+			(font
+				(size 1.48 1.48)
+			)
+			(justify left bottom)
+		)
+	)
+	(text "R10"
+		(exclude_from_sim no)
+		(at 80.01 114.704 90)
+		(effects
+			(font
+				(size 1.48 1.48)
+			)
+			(justify left top)
+		)
+	)
+	(text "10k"
+		(exclude_from_sim no)
+		(at 236.22 126.025 90)
+		(effects
+			(font
+				(size 1.48 1.48)
+			)
+			(justify left top)
+		)
+	)
+	(text "+20V"
+		(exclude_from_sim no)
+		(at 92.284 62.17 0)
+		(effects
+			(font
+				(size 1.48 1.48)
+			)
+			(justify left bottom)
+		)
+	)
+	(text "R6"
+		(exclude_from_sim no)
+		(at 115.621 83.82 0)
+		(effects
+			(font
+				(size 1.48 1.48)
+			)
+			(justify left top)
+		)
+	)
+	(text "5.1k"
+		(exclude_from_sim no)
+		(at 77.47 114.903 90)
+		(effects
+			(font
+				(size 1.48 1.48)
+			)
+			(justify left bottom)
+		)
+	)
+	(text "R7"
+		(exclude_from_sim no)
+		(at 115.584 96.52 0)
+		(effects
+			(font
+				(size 1.48 1.48)
+			)
+			(justify left top)
+		)
+	)
+	(text "C4"
+		(exclude_from_sim no)
+		(at 82.491 71.749 0)
+		(effects
+			(font
+				(size 1.48 1.48)
+			)
+			(justify left bottom)
+		)
+	)
+	(text "R11"
+		(exclude_from_sim no)
+		(at 90.17 114.377 90)
+		(effects
+			(font
+				(size 1.48 1.48)
+			)
+			(justify left top)
+		)
+	)
+	(text "U4"
+		(exclude_from_sim no)
+		(at 210.798 77.47 0)
+		(effects
+			(font
+				(size 1.48 1.48)
+			)
+			(justify left bottom)
+		)
+	)
+	(text "Q1"
+		(exclude_from_sim no)
+		(at 106.426 87.122 90)
+		(effects
+			(font
+				(size 1.48 1.48)
+			)
+			(justify left bottom)
+		)
+	)
+	(text "PD"
+		(exclude_from_sim no)
+		(at 230.584 102.856 90)
+		(effects
+			(font
+				(size 1.48 1.48)
+			)
+			(justify left bottom)
+		)
+	)
+	(text "C1"
+		(exclude_from_sim no)
+		(at 152.705 70.479 0)
+		(effects
+			(font
+				(size 1.48 1.48)
+			)
+			(justify left bottom)
+		)
+	)
+	(text "GND"
+		(exclude_from_sim no)
+		(at 196.082 114.3 0)
+		(effects
+			(font
+				(size 1.48 1.48)
+			)
+			(justify left bottom)
+		)
+	)
+	(text "100nF"
+		(exclude_from_sim no)
+		(at 150.65 74.301 0)
+		(effects
+			(font
+				(size 1.48 1.48)
+			)
+			(justify left top)
+		)
+	)
+	(text "5.1k"
+		(exclude_from_sim no)
+		(at 87.63 114.903 90)
+		(effects
+			(font
+				(size 1.48 1.48)
+			)
+			(justify left bottom)
+		)
+	)
+	(text "1k"
+		(exclude_from_sim no)
+		(at 116.021 81.28 0)
+		(effects
+			(font
+				(size 1.48 1.48)
+			)
+			(justify left bottom)
+		)
+	)
+	(text "10k"
+		(exclude_from_sim no)
+		(at 138.135 119.38 0)
+		(effects
+			(font
+				(size 1.48 1.48)
+			)
+			(justify left bottom)
+		)
+	)
+	(text "DMG7430LFG-7"
+		(exclude_from_sim no)
+		(at 93.726 92.71 90)
+		(effects
+			(font
+				(size 1.48 1.48)
+			)
+			(justify left top)
+		)
+	)
+	(text "5V"
+		(exclude_from_sim no)
+		(at 115.511 116.284 0)
+		(effects
+			(font
+				(size 1.48 1.48)
+			)
+			(justify left bottom)
+		)
+	)
+	(text "R5"
+		(exclude_from_sim no)
+		(at 233.68 125.716 90)
+		(effects
+			(font
+				(size 1.48 1.48)
+			)
+			(justify left bottom)
+		)
+	)
+	(text "J1"
+		(exclude_from_sim no)
+		(at 51.816 88.9 0)
+		(effects
+			(font
+				(size 1.48 1.48)
+			)
+			(justify left bottom)
+		)
+	)
+	(text "R9"
+		(exclude_from_sim no)
+		(at 138.48 121.92 0)
+		(effects
+			(font
+				(size 1.48 1.48)
+			)
+			(justify left top)
+		)
+	)
 	(junction
 		(at 69.85 95.25)
@@
 		)
 	)
-	(text "0.01"
-		(exclude_from_sim no)
-		(at 114.857 93.98 0)
-		(effects
-			(font
-				(size 1.48 1.48)
-			)
-			(justify left bottom)
-		)
-	)
-	(text "R10"
-		(exclude_from_sim no)
-		(at 80.01 114.704 90)
-		(effects
-			(font
-				(size 1.48 1.48)
-			)
-			(justify left top)
-		)
-	)
-	(text "10k"
-		(exclude_from_sim no)
-		(at 236.22 126.025 90)
-		(effects
-			(font
-				(size 1.48 1.48)
-			)
-			(justify left top)
-		)
-	)
-	(text "+20V"
-		(exclude_from_sim no)
-		(at 92.284 62.17 0)
-		(effects
-			(font
-				(size 1.48 1.48)
-			)
-			(justify left bottom)
-		)
-	)
-	(text "R6"
-		(exclude_from_sim no)
-		(at 115.621 83.82 0)
-		(effects
-			(font
-				(size 1.48 1.48)
-			)
-			(justify left top)
-		)
-	)
-	(text "5.1k"
-		(exclude_from_sim no)
-		(at 77.47 114.903 90)
-		(effects
-			(font
-				(size 1.48 1.48)
-			)
-			(justify left bottom)
-		)
-	)
-	(text "R7"
-		(exclude_from_sim no)
-		(at 115.584 96.52 0)
-		(effects
-			(font
-				(size 1.48 1.48)
-			)
-			(justify left top)
-		)
-	)
-	(text "C4"
-		(exclude_from_sim no)
-		(at 82.491 71.749 0)
-		(effects
-			(font
-				(size 1.48 1.48)
-			)
-			(justify left bottom)
-		)
-	)
-	(text "R11"
-		(exclude_from_sim no)
-		(at 90.17 114.377 90)
-		(effects
-			(font
-				(size 1.48 1.48)
-			)
-			(justify left top)
-		)
-	)
-	(text "U4"
-		(exclude_from_sim no)
-		(at 210.798 77.47 0)
-		(effects
-			(font
-				(size 1.48 1.48)
-			)
-			(justify left bottom)
-		)
-	)
-	(text "Q1"
-		(exclude_from_sim no)
-		(at 106.426 87.122 90)
-		(effects
-			(font
-				(size 1.48 1.48)
-			)
-			(justify left bottom)
-		)
-	)
-	(text "PD"
-		(exclude_from_sim no)
-		(at 230.584 102.856 90)
-		(effects
-			(font
-				(size 1.48 1.48)
-			)
-			(justify left bottom)
-		)
-	)
-	(text "C1"
-		(exclude_from_sim no)
-		(at 152.705 70.479 0)
-		(effects
-			(font
-				(size 1.48 1.48)
-			)
-			(justify left bottom)
-		)
-	)
-	(text "GND"
-		(exclude_from_sim no)
-		(at 196.082 114.3 0)
-		(effects
-			(font
-				(size 1.48 1.48)
-			)
-			(justify left bottom)
-		)
-	)
-	(text "100nF"
-		(exclude_from_sim no)
-		(at 150.65 74.301 0)
-		(effects
-			(font
-				(size 1.48 1.48)
-			)
-			(justify left top)
-		)
-	)
-	(text "5.1k"
-		(exclude_from_sim no)
-		(at 87.63 114.903 90)
-		(effects
-			(font
-				(size 1.48 1.48)
-			)
-			(justify left bottom)
-		)
-	)
-	(text "1k"
-		(exclude_from_sim no)
-		(at 116.021 81.28 0)
-		(effects
-			(font
-				(size 1.48 1.48)
-			)
-			(justify left bottom)
-		)
-	)
-	(text "10k"
-		(exclude_from_sim no)
-		(at 138.135 119.38 0)
-		(effects
-			(font
-				(size 1.48 1.48)
-			)
-			(justify left bottom)
-		)
-	)
-	(text "DMG7430LFG-7"
-		(exclude_from_sim no)
-		(at 93.726 92.71 90)
-		(effects
-			(font
-				(size 1.48 1.48)
-			)
-			(justify left top)
-		)
-	)
-	(text "5V"
-		(exclude_from_sim no)
-		(at 115.511 116.284 0)
-		(effects
-			(font
-				(size 1.48 1.48)
-			)
-			(justify left bottom)
-		)
-	)
-	(text "R5"
-		(exclude_from_sim no)
-		(at 233.68 125.716 90)
-		(effects
-			(font
-				(size 1.48 1.48)
-			)
-			(justify left bottom)
-		)
-	)
-	(text "J1"
-		(exclude_from_sim no)
-		(at 51.816 88.9 0)
-		(effects
-			(font
-				(size 1.48 1.48)
-			)
-			(justify left bottom)
-		)
-	)
-	(text "R9"
-		(exclude_from_sim no)
-		(at 138.48 121.92 0)
-		(effects
-			(font
-				(size 1.48 1.48)
-			)
-			(justify left top)
-		)
-	)

Commit message: Down-sized a bunch of resistor packags
Parts:
- R10, R11, R5, R9: footprint Resistor_SMD:R_0805_2012Metric -> Resistor_SMD:R_0603_1608Metric
Changed lines of the file:
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@@
 			)
 		)
-		(property "Footprint" "Resistor_SMD:R_0805_2012Metric"
+		(property "Footprint" "Resistor_SMD:R_0603_1608Metric"
 			(at 139.7 120.65 0)
 			(effects
@@
 			)
 		)
-		(property "Footprint" "Resistor_SMD:R_0805_2012Metric"
+		(property "Footprint" "Resistor_SMD:R_0603_1608Metric"
 			(at 234.95 124.46 0)
 			(effects
@@
 			)
 		)
-		(property "Footprint" "Resistor_SMD:R_0805_2012Metric"
+		(property "Footprint" "Resistor_SMD:R_0603_1608Metric"
 			(at 88.9 113.03 0)
 			(effects
@@
 			)
 		)
-		(property "Footprint" "Resistor_SMD:R_0805_2012Metric"
+		(property "Footprint" "Resistor_SMD:R_0603_1608Metric"
 			(at 78.74 113.03 0)
 			(effects
