File: ClockController.X/Hardware/rtc.kicad_sch (KiCad schematic)
At the start: 2 parts, among them Y1 RV-3028-C7_32.768KHZ_1PPM-TA-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

Commit message: Added missing footprint assignment
Parts:
- BT1: footprint (none) -> Battery_Holder_:BAT_BAT-HLD-003-SMT
Changed lines of the file:
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@@
 			)
 		)
-		(property "Footprint" ""
+		(property "Footprint" "Battery_Holder_:BAT_BAT-HLD-003-SMT"
 			(at 181.356 81.28 90)
 			(effects

Commit message: Converting to single board layout
Connections:
- net Batt Power: now reaches BT1.1 (+), Y1.6 (VBACKUP)
- net 5V renamed VDD
Other:
- moved on the sheet: BT1, Y1
Changed lines of the file:
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@@
 	(paper "USLetter")
 	(no_connect
-		(at 127 76.2)
+		(at 109.22 91.44)
 	)
 	(no_connect
-		(at 127 78.74)
+		(at 109.22 93.98)
 	)
 	(no_connect
-		(at 162.56 76.2)
+		(at 144.78 91.44)
 	)
 	(wire
 		(pts
-			(xy 162.56 81.28) (xy 177.8 81.28)
+			(xy 144.78 96.52) (xy 160.02 96.52)
 		)
 		(stroke
@@
 		)
 	)
-	(hierarchical_label "5V"
-		(shape input)
-		(at 162.56 78.74 0)
+	(label "Batt Power"
+		(at 149.86 96.52 0)
 		(effects
 			(font
 				(size 1.27 1.27)
 			)
-			(justify left)
-		)
-	)
-	(hierarchical_label "SCL"
-		(shape bidirectional)
-		(at 127 81.28 180)
+			(justify left bottom)
+		)
+	)
+	(hierarchical_label "VDD"
+		(shape input)
+		(at 144.78 93.98 0)
 		(effects
 			(font
 				(size 1.27 1.27)
 			)
-			(justify right)
-		)
-	)
-	(hierarchical_label "SDA"
+			(justify left)
+		)
+	)
+	(hierarchical_label "SCL"
 		(shape bidirectional)
-		(at 127 83.82 180)
+		(at 109.22 96.52 180)
 		(effects
 			(font
@@
 		)
 	)
+	(hierarchical_label "SDA"
+		(shape bidirectional)
+		(at 109.22 99.06 180)
+		(effects
+			(font
+				(size 1.27 1.27)
+			)
+			(justify right)
+		)
+	)
 	(symbol
 		(lib_id "power:GND")
-		(at 185.42 81.28 90)
+		(at 167.64 96.52 90)
 		(unit 1)
 		(exclude_from_sim no)
@@
 		(fields_autoplaced yes)
 		(property "Reference" "#PWR031"
-			(at 191.77 81.28 0)
+			(at 173.99 96.52 0)
 			(effects
 				(font
@@
 		)
 		(property "Value" "GND"
-			(at 189.23 81.2799 90)
+			(at 171.45 96.5199 90)
 			(effects
 				(font
@@
 		)
 		(property "Footprint" ""
-			(at 185.42 81.28 0)
+			(at 167.64 96.52 0)
 			(effects
 				(font
@@
 		)
 		(property "Datasheet" ""
-			(at 185.42 81.28 0)
+			(at 167.64 96.52 0)
 			(effects
 				(font
@@
 		)
 		(property "Description" "Power symbol creates a global label with name \"GND\" , ground"
-			(at 185.42 81.28 0)
+			(at 167.64 96.52 0)
 			(effects
 				(font
@@
 	(symbol
 		(lib_id "RTC_:RV-3028-C7_32.768KHZ_1PPM-TA-QC")
-		(at 127 76.2 0)
+		(at 109.22 91.44 0)
 		(unit 1)
 		(exclude_from_sim no)
@@
 		(fields_autoplaced yes)
 		(property "Reference" "Y1"
-			(at 144.78 68.58 0)
+			(at 127 83.82 0)
 			(effects
 				(font
@@
 		)
 		(property "Value" "RV-3028-C7_32.768KHZ_1PPM-TA-QC"
-			(at 144.78 71.12 0)
+			(at 127 86.36 0)
 			(effects
 				(font
@@
 		)
 		(property "Footprint" "RTC_:RV3028C732768KHZ1PPMTAQC"
-			(at 158.75 171.12 0)
+			(at 140.97 186.36 0)
 			(effects
 				(font
@@
 		)
 		(property "Datasheet" "https://www.microcrystal.com/fileadmin/Media/Products/RTC/Datasheet/RV-3028-C7.pdf"
-			(at 158.75 271.12 0)
+			(at 140.97 286.36 0)
 			(effects
 				(font
@@
 		)
 		(property "Description" "IC RTC CLK/CALENDAR I2C 8-SMT"
-			(at 127 76.2 0)
+			(at 109.22 91.44 0)
 			(effects
 				(font
@@
 		)
 		(property "Height" "0.8"
-			(at 158.75 471.12 0)
+			(at 140.97 486.36 0)
 			(effects
 				(font
@@
 		)
 		(property "Manufacturer_Name" "Micro Crystal AG"
-			(at 158.75 571.12 0)
+			(at 140.97 586.36 0)
 			(effects
 				(font
@@
 		)
 		(property "Manufacturer_Part_Number" "RV-3028-C7 32.768KHZ 1PPM-TA-QC"
-			(at 158.75 671.12 0)
+			(at 140.97 686.36 0)
 			(effects
 				(font
@@
 		)
 		(property "Mouser Part Number" ""
-			(at 158.75 771.12 0)
+			(at 140.97 786.36 0)
 			(effects
 				(font
@@
 		)
 		(property "Mouser Price/Stock" ""
-			(at 158.75 871.12 0)
+			(at 140.97 886.36 0)
 			(effects
 				(font
@@
 		)
 		(property "Arrow Part Number" ""
-			(at 158.75 971.12 0)
+			(at 140.97 986.36 0)
 			(effects
 				(font
@@
 		)
 		(property "Arrow Price/Stock" ""
-			(at 158.75 1071.12 0)
+			(at 140.97 1086.36 0)
 			(effects
 				(font
@@
 	(symbol
 		(lib_id "power:GND")
-		(at 162.56 83.82 90)
+		(at 144.78 99.06 90)
 		(unit 1)
 		(exclude_from_sim no)
@@
 		(fields_autoplaced yes)
 		(property "Reference" "#PWR030"
-			(at 168.91 83.82 0)
+			(at 151.13 99.06 0)
 			(effects
 				(font
@@
 		)
 		(property "Value" "GND"
-			(at 166.37 83.8199 90)
+			(at 148.59 99.0599 90)
 			(effects
 				(font
@@
 		)
 		(property "Footprint" ""
-			(at 162.56 83.82 0)
+			(at 144.78 99.06 0)
 			(effects
 				(font
@@
 		)
 		(property "Datasheet" ""
-			(at 162.56 83.82 0)
+			(at 144.78 99.06 0)
 			(effects
 				(font
@@
 		)
 		(property "Description" "Power symbol creates a global label with name \"GND\" , ground"
-			(at 162.56 83.82 0)
+			(at 144.78 99.06 0)
 			(effects
 				(font
@@
 	(symbol
 		(lib_id "Device:Battery_Cell")
-		(at 182.88 81.28 90)
+		(at 165.1 96.52 90)
 		(unit 1)
 		(exclude_from_sim no)
@@
 		(fields_autoplaced yes)
 		(property "Reference" "BT1"
-			(at 181.0385 73.66 90)
+			(at 163.2585 88.9 90)
 			(effects
 				(font
@@
 		)
 		(property "Value" "Battery_Cell"
-			(at 181.0385 76.2 90)
+			(at 163.2585 91.44 90)
 			(effects
 				(font
@@
 		)
 		(property "Footprint" "Battery_Holder_:BAT_BAT-HLD-003-SMT"
-			(at 181.356 81.28 90)
+			(at 163.576 96.52 90)
 			(effects
 				(font
@@
 		)
 		(property "Datasheet" "~"
-			(at 181.356 81.28 90)
+			(at 163.576 96.52 90)
 			(effects
 				(font
@@
 		)
 		(property "Description" "Single-cell battery"
-			(at 182.88 81.28 0)
+			(at 165.1 96.52 0)
 			(effects
 				(font
@@
 		)
 		(property "Sim.Device" "V"
-			(at 182.88 81.28 0)
+			(at 165.1 96.52 0)
 			(effects
 				(font
@@
 		)
 		(property "Sim.Type" "DC"
-			(at 182.88 81.28 0)
+			(at 165.1 96.52 0)
 			(effects
 				(font
@@
 		)
 		(property "Sim.Pins" "1=+ 2=-"
-			(at 182.88 81.28 0)
-			(effects
-				(font
+			(at 165.1 96.52 0)
+			(effects
+				(font
