File: ClockController.X/Hardware/+5 VRC.kicad_sch (KiCad schematic)
At the start: 4 parts, among them U2 AS78L05RTR-E1

Commit message: Updated most footprints
Parts:
- C5, C6: footprint Clock Controller:CAP_0805 -> Capacitor_SMD:C_0805_2012Metric
- U2: footprint Clock Controller:DIODES_SOT89 -> Package_TO_SOT_SMD:SOT-89-3
Changed lines of the file:
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@@
 			)
 		)
-		(property "Footprint" "Clock Controller:CAP_0805"
+		(property "Footprint" "Capacitor_SMD:C_0805_2012Metric"
 			(at 187.96 111.76 0)
 			(effects
@@
 			)
 		)
-		(property "Footprint" "Clock Controller:CAP_0805"
+		(property "Footprint" "Capacitor_SMD:C_0805_2012Metric"
 			(at 119.38 113.03 0)
 			(effects
@@
 			)
 		)
-		(property "Footprint" "Clock Controller:DIODES_SOT89"
+		(property "Footprint" "Package_TO_SOT_SMD:SOT-89-3"
 			(at 124.46 104.14 0)
 			(effects

Commit message: Replacing many thin traces with poured zones.
Changed lines of the file:
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@@
 (kicad_sch
-	(version 20231120)
+	(version 20250114)
 	(generator "eeschema")
-	(generator_version "8.0")
+	(generator_version "9.0")
 	(paper "A4")
+	(text "+20V"
+		(exclude_from_sim no)
+		(at 184.994 92.65 0)
+		(effects
+			(font
+				(size 1.48 1.48)
+			)
+			(justify left bottom)
+		)
+	)
+	(text "C6"
+		(exclude_from_sim no)
+		(at 186.049 113.015 90)
+		(effects
+			(font
+				(size 1.48 1.48)
+			)
+			(justify left bottom)
+		)
+	)
+	(text "Vcc"
+		(exclude_from_sim no)
+		(at 98.401 93.345 0)
+		(effects
+			(font
+				(size 1.48 1.48)
+			)
+			(justify left bottom)
+		)
+	)
+	(text "C5"
+		(exclude_from_sim no)
+		(at 117.469 114.322 90)
+		(effects
+			(font
+				(size 1.48 1.48)
+			)
+			(justify left bottom)
+		)
+	)
+	(text "U2"
+		(exclude_from_sim no)
+		(at 123.204 97.79 0)
+		(effects
+			(font
+				(size 1.48 1.48)
+			)
+			(justify left bottom)
+		)
+	)
+	(text "+5V"
+		(exclude_from_sim no)
+		(at 117.16 92.65 0)
+		(effects
+			(font
+				(size 1.48 1.48)
+			)
+			(justify left bottom)
+		)
+	)
 	(junction
 		(at 119.38 104.14)
@@
 		)
 	)
-	(text "+20V"
-		(exclude_from_sim no)
-		(at 184.994 92.65 0)
-		(effects
-			(font
-				(size 1.48 1.48)
-			)
-			(justify left bottom)
-		)
-	)
-	(text "C6"
-		(exclude_from_sim no)
-		(at 186.049 113.015 90)
-		(effects
-			(font
-				(size 1.48 1.48)
-			)
-			(justify left bottom)
-		)
-	)
-	(text "Vcc"
-		(exclude_from_sim no)
-		(at 98.401 93.345 0)
-		(effects
-			(font
-				(size 1.48 1.48)
-			)
-			(justify left bottom)
-		)
-	)
-	(text "C5"
-		(exclude_from_sim no)
-		(at 117.469 114.322 90)
-		(effects
-			(font
-				(size 1.48 1.48)
-			)
-			(justify left bottom)
-		)
-	)
-	(text "U2"
-		(exclude_from_sim no)
-		(at 123.204 97.79 0)
-		(effects
-			(font
-				(size 1.48 1.48)
-			)
-			(justify left bottom)
-		)
-	)
-	(text "+5V"
-		(exclude_from_sim no)
-		(at 117.16 92.65 0)
-		(effects
-			(font
-				(size 1.48 1.48)
-			)
-			(justify left bottom)
-		)
-	)
