File: Hardware/Nixie Driver Tester/Boost Converter.kicad_sch (KiCad schematic)
At the start: 6 parts, among them Q1 MMBT2222A, Q2 MMBT2907ALT1G, Q3 FDD7N25LZTM

Commit message: First reasonable layout.
Parts:
- C2: footprint Capacitor_SMD:C_0603_1608Metric -> Capacitor_SMD:C_0805_2012Metric
Changed lines of the file:
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@@
 			)
 		)
-		(property "Footprint" "Capacitor_SMD:C_0603_1608Metric"
+		(property "Footprint" "Capacitor_SMD:C_0805_2012Metric"
 			(at 153.3652 92.71 0)
 			(effects
