File: Hardware/Nixie Driver Tester/USB PD.kicad_sch (KiCad schematic)
At the start: 6 parts, among them J2 UJC-HP-3-SMT-TR

Commit message: Initial component layout.
Parts:
- R6, R7, R8: footprint Resistor_SMD:R_0201_0603Metric -> Resistor_SMD:R_0603_1608Metric
Connections:
- net GND: no longer U2.4 (CC1), U2.5 (CC2)
- net CC1: now reaches J2.A5 (CC1), R6.2
- net CC1: now also U2.4 (CC1)
- net CC2: now reaches J2.B5 (CC2), R7.1
- net CC2: now also U2.5 (CC2)
Other:
- moved on the sheet: R6, R7
Changed lines of the file:
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@@
-	(wire
-		(pts
-			(xy 181.61 52.07) (xy 173.99 52.07)
-		)
-		(stroke
-			(width 0)
-			(type default)
-		)
-	)
 	(wire
 		(pts
@@
 	(wire
 		(pts
-			(xy 181.61 49.53) (xy 173.99 49.53)
+			(xy 180.34 49.53) (xy 181.61 49.53)
 		)
 		(stroke
@@
 	(wire
 		(pts
-			(xy 160.02 49.53) (xy 166.37 49.53)
-		)
-		(stroke
-			(width 0)
-			(type default)
-		)
-	)
-	(wire
-		(pts
-			(xy 160.02 52.07) (xy 166.37 52.07)
+			(xy 160.02 49.53) (xy 172.72 49.53)
+		)
+		(stroke
+			(width 0)
+			(type default)
+		)
+	)
+	(wire
+		(pts
+			(xy 160.02 52.07) (xy 172.72 52.07)
 		)
 		(stroke
@@
 		(pts
 			(xy 132.08 54.61) (xy 127 54.61)
+		)
+		(stroke
+			(width 0)
+			(type default)
+		)
+	)
+	(wire
+		(pts
+			(xy 180.34 52.07) (xy 181.61 52.07)
 		)
 		(stroke
@@
 	)
 	(label "CC1"
-		(at 179.07 49.53 90)
+		(at 170.18 49.53 90)
 		(fields_autoplaced yes)
 		(effects
@@
 	)
 	(label "CC2"
-		(at 179.07 52.07 270)
+		(at 170.18 52.07 270)
 		(fields_autoplaced yes)
 		(effects
@@
 	(symbol
 		(lib_id "Device:R_US")
-		(at 170.18 49.53 270)
+		(at 176.53 49.53 270)
 		(mirror x)
 		(unit 1)
@@
 		(dnp no)
 		(property "Reference" "R6"
-			(at 171.4501 46.99 0)
+			(at 177.8001 46.99 0)
 			(effects
 				(font
@@
 		)
 		(property "Value" "5.1k"
-			(at 168.9101 46.99 0)
+			(at 175.2601 46.99 0)
 			(effects
 				(font
@@
 			)
 		)
-		(property "Footprint" "Resistor_SMD:R_0201_0603Metric"
-			(at 169.926 48.514 90)
+		(property "Footprint" "Resistor_SMD:R_0603_1608Metric"
+			(at 176.276 48.514 90)
 			(effects
 				(font
@@
 		)
 		(property "Datasheet" "~"
-			(at 170.18 49.53 0)
+			(at 176.53 49.53 0)
 			(effects
 				(font
@@
 		)
 		(property "Description" "Resistor, US symbol"
-			(at 170.18 49.53 0)
+			(at 176.53 49.53 0)
 			(effects
 				(font
@@
 			)
 		)
-		(property "Footprint" "Resistor_SMD:R_0201_0603Metric"
+		(property "Footprint" "Resistor_SMD:R_0603_1608Metric"
 			(at 171.704 87.884 90)
 			(effects
@@
 	(symbol
 		(lib_id "Device:R_US")
-		(at 170.18 52.07 90)
+		(at 176.53 52.07 90)
 		(mirror x)
 		(unit 1)
@@
 		(dnp no)
 		(property "Reference" "R7"
-			(at 168.9099 54.61 0)
+			(at 175.2599 54.61 0)
 			(effects
 				(font
@@
 		)
 		(property "Value" "5.1k"
-			(at 171.4499 54.61 0)
+			(at 177.7999 54.61 0)
 			(effects
 				(font
@@
 			)
 		)
-		(property "Footprint" "Resistor_SMD:R_0201_0603Metric"
-			(at 170.434 53.086 90)
+		(property "Footprint" "Resistor_SMD:R_0603_1608Metric"
+			(at 176.784 53.086 90)
 			(effects
 				(font
@@
 		)
 		(property "Datasheet" "~"
-			(at 170.18 52.07 0)
+			(at 176.53 52.07 0)
 			(effects
 				(font
@@
 		)
 		(property "Description" "Resistor, US symbol"
-			(at 170.18 52.07 0)
-			(effects
-				(font
+			(at 176.53 52.07 0)
+			(effects
+				(font

Commit message: First reasonable layout.
Connections:
- net VBUS: now also S1.1, S1.6; no longer J2.A9 (V-BUS_1), J2.B9 (V-BUS_2), S1.2, S1.5
- new net VBUS In: J2.A9 (V-BUS_1), J2.B9 (V-BUS_2), S1.2, S1.5, U2.1 (VIN)
Other:
- moved on the sheet: R8, U2
Changed lines of the file:
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@@
 	)
 	(junction
-		(at 127 83.82)
-		(diameter 0)
-		(color 0 0 0 0)
-	)
-	(junction
-		(at 163.83 46.99)
+		(at 120.65 83.82)
 		(diameter 0)
 		(color 0 0 0 0)
@@
 	)
 	(no_connect
-		(at 134.62 88.9)
+		(at 152.4 96.52)
 	)
 	(no_connect
@@
 	)
 	(no_connect
-		(at 157.48 83.82)
+		(at 175.26 91.44)
 	)
 	(no_connect
-		(at 134.62 86.36)
+		(at 152.4 93.98)
 	)
 	(no_connect
@@
 	(wire
 		(pts
-			(xy 157.48 88.9) (xy 167.64 88.9)
+			(xy 175.26 96.52) (xy 185.42 96.52)
 		)
 		(stroke
@@
 	(wire
 		(pts
-			(xy 101.6 114.3) (xy 127 114.3)
-		)
-		(stroke
-			(width 0)
-			(type default)
-		)
-	)
-	(wire
-		(pts
-			(xy 101.6 83.82) (xy 127 83.82)
+			(xy 101.6 114.3) (xy 120.65 114.3)
+		)
+		(stroke
+			(width 0)
+			(type default)
+		)
+	)
+	(wire
+		(pts
+			(xy 101.6 83.82) (xy 120.65 83.82)
 		)
 		(stroke
@@
 	(wire
 		(pts
-			(xy 127 83.82) (xy 127 114.3)
+			(xy 120.65 83.82) (xy 120.65 114.3)
 		)
 		(stroke
@@
 	(wire
 		(pts
-			(xy 127 83.82) (xy 134.62 83.82)
-		)
-		(stroke
-			(width 0)
-			(type default)
-		)
-	)
-	(wire
-		(pts
 			(xy 160.02 54.61) (xy 163.83 54.61)
 		)
@@
 	(wire
 		(pts
-			(xy 163.83 41.91) (xy 163.83 46.99)
+			(xy 120.65 78.74) (xy 120.65 83.82)
 		)
 		(stroke
@@
 	(text_box "10ohms on VSET selects the 12V PDO."
 		(exclude_from_sim no)
-		(at 170.18 93.98 0)
+		(at 187.96 101.6 0)
 		(size 22.86 5.08)
 		(stroke
@@
 	)
 	(label "CC2"
-		(at 134.62 93.98 180)
+		(at 152.4 101.6 180)
 		(fields_autoplaced yes)
 		(effects
@@
 		)
 	)
-	(label "VBUS"
-		(at 99.06 115.57 270)
+	(label "VBUS In"
+		(at 152.4 91.44 180)
 		(fields_autoplaced yes)
 		(effects
@@
 		)
 	)
-	(label "CC1"
-		(at 134.62 91.44 180)
+	(label "VBUS In"
+		(at 99.06 115.57 270)
 		(fields_autoplaced yes)
 		(effects
@@
 		)
 	)
-	(label "VBUS"
-		(at 99.06 82.55 90)
+	(label "CC1"
+		(at 152.4 99.06 180)
 		(fields_autoplaced yes)
 		(effects
@@
 				(size 1.27 1.27)
 			)
-			(justify left)
-		)
-	)
-	(label "VBUS"
-		(at 163.83 54.61 270)
+			(justify right)
+		)
+	)
+	(label "VBUS In"
+		(at 99.06 82.55 90)
 		(fields_autoplaced yes)
 		(effects
@@
 				(size 1.27 1.27)
 			)
-			(justify right bottom)
-		)
-	)
-	(label "CC2"
-		(at 170.18 52.07 270)
+			(justify left)
+		)
+	)
+	(label "VBUS In"
+		(at 163.83 54.61 270)
 		(fields_autoplaced yes)
 		(effects
@@
 		)
 	)
-	(hierarchical_label "SDA"
-		(shape bidirectional)
-		(at 157.48 93.98 0)
+	(label "CC2"
+		(at 170.18 52.07 270)
 		(fields_autoplaced yes)
 		(effects
@@
 				(size 1.27 1.27)
 			)
-			(justify left)
-		)
-	)
-	(hierarchical_label "SCL"
+			(justify right bottom)
+		)
+	)
+	(hierarchical_label "SDA"
 		(shape bidirectional)
-		(at 157.48 91.44 0)
+		(at 175.26 101.6 0)
 		(fields_autoplaced yes)
 		(effects
@@
 		)
 	)
+	(hierarchical_label "SCL"
+		(shape bidirectional)
+		(at 175.26 99.06 0)
+		(fields_autoplaced yes)
+		(effects
+			(font
+				(size 1.27 1.27)
+			)
+			(justify left)
+		)
+	)
 	(hierarchical_label "VBUS"
 		(shape output)
-		(at 163.83 41.91 90)
+		(at 120.65 78.74 90)
 		(fields_autoplaced yes)
 		(effects
@@
 	(symbol
 		(lib_id "power:GND")
-		(at 175.26 88.9 90)
+		(at 193.04 96.52 90)
 		(unit 1)
 		(exclude_from_sim no)
@@
 		(fields_autoplaced yes)
 		(property "Reference" "#PWR08"
-			(at 181.61 88.9 0)
+			(at 199.39 96.52 0)
 			(effects
 				(font
@@
 		)
 		(property "Value" "GND"
-			(at 179.07 88.8999 90)
+			(at 196.85 96.5199 90)
 			(effects
 				(font
@@
 		)
 		(property "Footprint" ""
-			(at 175.26 88.9 0)
+			(at 193.04 96.52 0)
 			(effects
 				(font
@@
 		)
 		(property "Datasheet" ""
-			(at 175.26 88.9 0)
+			(at 193.04 96.52 0)
 			(effects
 				(font
@@
 		)
 		(property "Description" "Power symbol creates a global label with name \"GND\" , ground"
-			(at 175.26 88.9 0)
+			(at 193.04 96.52 0)
 			(effects
 				(font
@@
 	(symbol
 		(lib_id "power:GND")
-		(at 157.48 86.36 90)
+		(at 175.26 93.98 90)
 		(unit 1)
 		(exclude_from_sim no)
@@
 		(fields_autoplaced yes)
 		(property "Reference" "#PWR07"
-			(at 163.83 86.36 0)
+			(at 181.61 93.98 0)
 			(effects
 				(font
@@
 		)
 		(property "Value" "GND"
-			(at 161.29 86.3599 90)
+			(at 179.07 93.9799 90)
 			(effects
 				(font
@@
 		)
 		(property "Footprint" ""
-			(at 157.48 86.36 0)
+			(at 175.26 93.98 0)
 			(effects
 				(font
@@
 		)
 		(property "Datasheet" ""
-			(at 157.48 86.36 0)
+			(at 175.26 93.98 0)
 			(effects
 				(font
@@
 		)
 		(property "Description" "Power symbol creates a global label with name \"GND\" , ground"
-			(at 157.48 86.36 0)
+			(at 175.26 93.98 0)
 			(effects
 				(font
@@
 	(symbol
 		(lib_id "Device:R_US")
-		(at 171.45 88.9 90)
+		(at 189.23 96.52 90)
 		(unit 1)
 		(exclude_from_sim no)
@@
 		(dnp no)
 		(property "Reference" "R8"
-			(at 171.45 86.36 90)
+			(at 189.23 93.98 90)
 			(effects
 				(font
@@
 		)
 		(property "Value" "10"
-			(at 171.45 91.44 90)
+			(at 189.23 99.06 90)
 			(effects
 				(font
@@
 		)
 		(property "Footprint" "Resistor_SMD:R_0603_1608Metric"
-			(at 171.704 87.884 90)
+			(at 189.484 95.504 90)
 			(effects
 				(font
@@
 		)
 		(property "Datasheet" "~"
-			(at 171.45 88.9 0)
+			(at 189.23 96.52 0)
 			(effects
 				(font
@@
 		)
 		(property "Description" "Resistor, US symbol"
-			(at 171.45 88.9 0)
+			(at 189.23 96.52 0)
 			(effects
 				(font
@@
 	(symbol
 		(lib_id "Interface_USB_:HUSB238")
-		(at 146.05 88.9 0)
+		(at 163.83 96.52 0)
 		(unit 1)
 		(exclude_from_sim no)
@@
 		(fields_autoplaced yes)
 		(property "Reference" "U2"
-			(at 146.05 78.74 0)
+			(at 163.83 86.36 0)
 			(effects
 				(font
@@
 		)
 		(property "Value" "~"
-			(at 146.05 88.9 0)
+			(at 163.83 96.52 0)
 			(effects
 				(font
@@
 		)
 		(property "Footprint" "Package_DFN_QFN:DFN-10-1EP_3x3mm_P0.5mm_EP1.65x2.38mm"
-			(at 146.05 88.9 0)
+			(at 163.83 96.52 0)
 			(effects
 				(font
@@
 		)
 		(property "Datasheet" ""
-			(at 146.05 88.9 0)
+			(at 163.83 96.52 0)
 			(effects
 				(font
@@
 		)
 		(property "Description" ""
-			(at 146.05 88.9 0)
+			(at 163.83 96.52 0)
 			(effects
 				(font
@@
 	(symbol
 		(lib_id "power:GND")
-		(at 146.05 99.06 0)
+		(at 163.83 106.68 0)
 		(unit 1)
 		(exclude_from_sim no)
@@
 		(fields_autoplaced yes)
 		(property "Reference" "#PWR05"
-			(at 146.05 105.41 0)
+			(at 163.83 113.03 0)
 			(effects
 				(font
@@
 		)
 		(property "Value" "GND"
-			(at 146.05 104.14 0)
+			(at 163.83 111.76 0)
 			(effects
 				(font
@@
 		)
 		(property "Footprint" ""
-			(at 146.05 99.06 0)
+			(at 163.83 106.68 0)
 			(effects
 				(font
@@
 		)
 		(property "Datasheet" ""
-			(at 146.05 99.06 0)
+			(at 163.83 106.68 0)
 			(effects
 				(font
@@
 		)
 		(property "Description" "Power symbol creates a global label with name \"GND\" , ground"
-			(at 146.05 99.06 0)
-			(effects
-				(font
+			(at 163.83 106.68 0)
+			(effects
+				(font
