File: Hardware/Nixie Driver Tester/USB PD.kicad_sch (KiCad schematic)
At the start: 6 parts, among them J2 UJC-HP-3-SMT-TR

Commit message: Status LEDs and switch labels
Parts:
- added D2, D3: LED, LED_SMD:LED_0603_1608Metric, symbol Device:LED
- added R10, R9: 49k, Resistor_SMD:R_0603_1608Metric, symbol Device:R_US
Connections:
- net GND: now also R10.2, R9.2
- net VBUS: now also D2.2 (A)
- net VBUS In: now also D3.2 (A)
- new net: D2.1 (K), R10.1
- new net: D3.1 (K), R9.1
