File: Hardware/Nixie Driver Tester/USB PD.kicad_sch (KiCad schematic)
At the start: 10 parts, among them J2 UJC-HP-3-SMT-TR

Commit message: No idea what I was working on here...
Other:
- moved on the sheet: D2, D3, R10, R9
