File: Hardware/Nixie Driver Tester/5V VRM.kicad_sch (KiCad schematic)
At the start: 3 parts

Commit message: First reasonable layout.
Parts:
- C6: value 100nF -> 1uF; footprint Capacitor_SMD:C_0603_1608Metric -> Capacitor_SMD:C_0805_2012Metric
Changed lines of the file:
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@@
 			)
 		)
-		(property "Value" "100nF"
+		(property "Value" "1uF"
 			(at 111.76 102.8699 0)
 			(effects
@@
 			)
 		)
-		(property "Footprint" "Capacitor_SMD:C_0603_1608Metric"
+		(property "Footprint" "Capacitor_SMD:C_0805_2012Metric"
 			(at 108.9152 105.41 0)
 			(effects
