File: Hardware/Nixie Driver Tester/Nixie Driver Tester.kicad_pcb (KiCad board)
At the start: 2 copper layers, 46.4 x 45.1 mm, 33 parts, among them J1 ICSP, J2 UJC-HP-3-SMT-TR, J3 OLED, Q1 MMBT2222A, Q2 MMBT2907ALT1G, Q3 FDD7N25LZTM, SW1 SW_Omron_B3FS

Commit message: No idea what I was working on here...
Parts:
- C2: footprint Capacitor_SMD:C_0805_2012Metric -> Resistor_SMD:R_1812_4532Metric
- S1: footprint SamacSys_Parts:SLW1116297AD -> Switch_:SLW1116297AD
- moved R6 28.3 mm to (160.0, 101.6), turned to 0 degrees
- moved H2 28.3 mm to (146.1, 82.5)
- moved R7 24.1 mm to (160.0, 96.5), turned to 180 degrees
- moved Q3 23.5 mm to (156.2, 84.5), turned to 0 degrees
- moved U2 22.4 mm to (158.3, 99.1), turned to 180 degrees
- moved H1 20.3 mm to (146.1, 108.6)
- moved D1 20.1 mm to (151.1, 84.3), turned to 90 degrees
- moved R8 19.9 mm to (155.4, 100.3), turned to -90 degrees
- moved S1 19.8 mm to (160.0, 109.2), turned to 0 degrees
- moved Q2 18.0 mm to (154.9, 93.0), turned to 180 degrees
- moved J2 17.4 mm to (163.2, 98.2), turned to 90 degrees
- moved C2 15.5 mm to (149.4, 88.9), turned to 180 degrees
- moved R10 15.3 mm to (154.2, 111.0), turned to -90 degrees
- moved D2 13.9 mm to (154.2, 108.0), turned to 90 degrees
- moved Q1 12.6 mm to (150.4, 93.0), turned to 180 degrees
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Routing:
- net /Boost Converter/PWM: track 16.2 -> 39.2 mm, vias 0 -> 2
- net GND: track 1.66 -> 21.7 mm, vias 0 -> 12
- net /5V VRM/VBUS: track 33.6 -> 47.0 mm, vias 0 -> 2
- net /5V VRM/5V: track 76.5 -> 64.7 mm, vias 3 -> 4
- net Net-(D1-A): track 23.2 -> 11.7 mm
- net /USB PD/CC1: track 17.7 -> 7.31 mm
- net Net-(R5-Pad2): track 27.5 -> 17.3 mm
- net /Button/Button: track 30.2 -> 40.2 mm, vias 2 -> 3
- net /USB PD/CC2: track 13.4 -> 5.25 mm, vias 2 -> 0
- net /Controller/SCL: track 52.1 -> 45.1 mm
- net /USB PD/VBUS In: track 31.7 -> 25.6 mm, vias 2 -> 0
- net /Controller/SDA: track 49.3 -> 45.3 mm
- net Net-(U2-VSET): track 3.89 -> 1.61 mm
- net Net-(D2-K): track 1.54 -> 0.00 mm
- net Net-(J1-Pin_5): track 17.5 -> 16.2 mm, vias 0 -> 1
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Other:
- board text added: "Nixie Driver Tester Aaron Johnson 02/09/2026"
- board text added: "On"
- board text added: "USB"
- board text removed: "Nixie Driver Tester Aaron Johnson 02/06/2025"
- board text removed: "◀ OFF ON ▶"
