File: Hardware/Nixie Driver Tester/Nixie.kicad_sch (KiCad schematic)
At the start: 1 part

Commit message: No idea what I was working on here...
Changed lines of the file:
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@@
+	(wire
+		(pts
+			(xy 172.72 81.28) (xy 165.1 81.28)
+		)
+		(stroke
+			(width 0)
+			(type default)
+		)
+	)
 	(wire
 		(pts
@@
 	(hierarchical_label "180V"
 		(shape input)
-		(at 165.1 81.28 0)
+		(at 172.72 81.28 0)
 		(effects
 			(font
@@
 		)
 	)
+	(netclass_flag ""
+		(length 2.54)
+		(shape round)
+		(at 168.91 81.28 180)
+		(fields_autoplaced yes)
+		(effects
+			(font
+				(size 1.27 1.27)
+			)
+			(justify right bottom)
+		)
+		(property "Netclass" "Thicc"
+			(at 169.6085 83.82 0)
+			(effects
+				(font
+					(size 1.27 1.27)
+				)
+				(justify left)
+			)
+		)
+		(property "Component Class" ""
+			(at -38.1 10.16 0)
+			(effects
+				(font
+					(size 1.27 1.27)
+					(italic yes)
+				)
+			)
+		)
+	)
