File: Hardware/Nixie Driver Tester/Nixie.kicad_sch (KiCad schematic)
At the start: 1 part

Commit message: New driver interface
Parts:
- added R9: 68, Resistor_SMD:R_1206_3216Metric, symbol Device:R_US
Connections:
- net 180V: now also N1.3 (Vnn); no longer N1.8 (Vnn)
- net 5V: now also N1.1 (Vdd); no longer N1.9 (Vdd)
- net GND: now also R9.2; no longer N1.10 (GND), N1.5 (ADDR2), N1.6 (ADDR1)
- net SCL: now also N1.5 (SCL); no longer N1.3 (SCL)
- net SDA: now also N1.6 (SDA); no longer N1.2 (SDA)
- new net: N1.2 (ADDR), R9.1
- no-connect marks 2 -> 0
Changed lines of the file:
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@@
 	(generator_version "10.0")
 	(paper "A4")
-	(junction
-		(at 153.67 96.52)
-		(diameter 0)
-		(color 0 0 0 0)
-	)
-	(junction
-		(at 151.13 96.52)
-		(diameter 0)
-		(color 0 0 0 0)
-	)
-	(no_connect
-		(at 156.21 93.98)
-	)
-	(no_connect
-		(at 139.7 76.2)
-	)
 	(wire
 		(pts
-			(xy 151.13 96.52) (xy 153.67 96.52)
+			(xy 153.67 100.33) (xy 153.67 93.98)
 		)
 		(stroke
@@
 	(wire
 		(pts
-			(xy 153.67 99.06) (xy 153.67 96.52)
-		)
-		(stroke
-			(width 0)
-			(type default)
-		)
-	)
-	(wire
-		(pts
-			(xy 172.72 81.28) (xy 165.1 81.28)
-		)
-		(stroke
-			(width 0)
-			(type default)
-		)
-	)
-	(wire
-		(pts
-			(xy 151.13 93.98) (xy 151.13 96.52)
-		)
-		(stroke
-			(width 0)
-			(type default)
-		)
-	)
-	(wire
-		(pts
-			(xy 148.59 93.98) (xy 148.59 96.52)
-		)
-		(stroke
-			(width 0)
-			(type default)
-		)
-	)
-	(wire
-		(pts
-			(xy 148.59 96.52) (xy 151.13 96.52)
-		)
-		(stroke
-			(width 0)
-			(type default)
-		)
-	)
-	(wire
-		(pts
-			(xy 153.67 96.52) (xy 153.67 93.98)
+			(xy 165.1 81.28) (xy 170.18 81.28)
 		)
 		(stroke
@@
 	(hierarchical_label "180V"
 		(shape input)
-		(at 172.72 81.28 0)
+		(at 153.67 100.33 270)
 		(effects
 			(font
 				(size 1.27 1.27)
 			)
-			(justify left)
+			(justify right)
 		)
 	)
@@
 		(length 2.54)
 		(shape round)
-		(at 168.91 81.28 180)
-		(fields_autoplaced yes)
+		(at 153.67 97.79 270)
 		(effects
 			(font
@@
 		)
 		(property "Netclass" "Thicc"
-			(at 169.6085 83.82 0)
+			(at 157.48 97.79 0)
 			(show_name no)
 			(do_not_autoplace no)
@@
 		)
 		(property "Component Class" ""
-			(at -38.1 10.16 0)
+			(at -53.34 26.67 0)
 			(show_name no)
 			(do_not_autoplace no)
@@
 	)
 	(symbol
-		(lib_id "power:GND")
-		(at 165.1 76.2 90)
+		(lib_id "Device:R_US")
+		(at 173.99 81.28 90)
 		(unit 1)
 		(body_style 1)
@@
 		(dnp no)
 		(fields_autoplaced yes)
-		(property "Reference" "#PWR027"
-			(at 171.45 76.2 0)
-			(hide yes)
-			(show_name no)
-			(do_not_autoplace no)
-			(effects
-				(font
-					(size 1.27 1.27)
-				)
-			)
-		)
-		(property "Value" "GND"
-			(at 168.91 76.1999 90)
-			(show_name no)
-			(do_not_autoplace no)
-			(effects
-				(font
-					(size 1.27 1.27)
-				)
-				(justify right)
-			)
-		)
-		(property "Footprint" ""
-			(at 165.1 76.2 0)
+		(property "Reference" "R9"
+			(at 173.99 74.93 90)
+			(show_name no)
+			(do_not_autoplace no)
+			(effects
+				(font
+					(size 1.27 1.27)
+				)
+			)
+		)
+		(property "Value" "68"
+			(at 173.99 77.47 90)
+			(show_name no)
+			(do_not_autoplace no)
+			(effects
+				(font
+					(size 1.27 1.27)
+				)
+			)
+		)
+		(property "Footprint" "Resistor_SMD:R_1206_3216Metric"
+			(at 174.244 80.264 90)
 			(hide yes)
 			(show_name no)
@@
 		)
 		(property "Datasheet" ""
-			(at 165.1 76.2 0)
-			(hide yes)
-			(show_name no)
-			(do_not_autoplace no)
-			(effects
-				(font
-					(size 1.27 1.27)
-				)
-			)
-		)
-		(property "Description" "Power symbol creates a global label with name \"GND\" , ground"
-			(at 165.1 76.2 0)
-			(hide yes)
-			(show_name no)
-			(do_not_autoplace no)
-			(effects
-				(font
-					(size 1.27 1.27)
-				)
-			)
+			(at 173.99 81.28 0)
+			(hide yes)
+			(show_name no)
+			(do_not_autoplace no)
+			(effects
+				(font
+					(size 1.27 1.27)
+				)
+			)
+		)
+		(property "Description" "Resistor, US symbol"
+			(at 173.99 81.28 0)
+			(hide yes)
+			(show_name no)
+			(do_not_autoplace no)
+			(effects
+				(font
+					(size 1.27 1.27)
+				)
+			)
+		)
+		(pin "2"
 		)
 		(pin "1"
@@
 			(project "Nixie Driver Tester"
 				(path "/c2082ee6-4c2e-4b3c-b2d7-410eae192cfe/394d8c35-7fb7-4f2e-9832-1fea7fce0352"
-					(reference "#PWR027")
+					(reference "R9")
 					(unit 1)
 				)
@@
 		(pin "5"
 		)
-		(pin "7"
-		)
-		(pin "8"
-		)
 		(pin "2"
 		)
-		(pin "9"
-		)
 		(pin "3"
-		)
-		(pin "10"
 		)
 		(instances
@@
 	(symbol
 		(lib_id "power:GND")
-		(at 153.67 99.06 0)
+		(at 151.13 93.98 0)
 		(unit 1)
 		(body_style 1)
@@
 		(fields_autoplaced yes)
 		(property "Reference" "#PWR026"
-			(at 153.67 105.41 0)
+			(at 151.13 100.33 0)
 			(hide yes)
 			(show_name no)
@@
 		)
 		(property "Value" "GND"
-			(at 153.67 104.14 0)
+			(at 151.13 99.06 0)
 			(show_name no)
 			(do_not_autoplace no)
@@
 		)
 		(property "Footprint" ""
-			(at 153.67 99.06 0)
+			(at 151.13 93.98 0)
 			(hide yes)
 			(show_name no)
@@
 		)
 		(property "Datasheet" ""
-			(at 153.67 99.06 0)
+			(at 151.13 93.98 0)
 			(hide yes)
 			(show_name no)
@@
 		)
 		(property "Description" "Power symbol creates a global label with name \"GND\" , ground"
-			(at 153.67 99.06 0)
+			(at 151.13 93.98 0)
 			(hide yes)
 			(show_name no)
@@
 					(unit 1)
 				)
+			)
+		)
+	)
+	(symbol
+		(lib_id "power:GND")
+		(at 177.8 81.28 90)
+		(unit 1)
+		(body_style 1)
+		(exclude_from_sim no)
+		(in_bom yes)
+		(on_board yes)
+		(in_pos_files yes)
+		(dnp no)
+		(fields_autoplaced yes)
+		(property "Reference" "#PWR027"
+			(at 184.15 81.28 0)
+			(hide yes)
+			(show_name no)
+			(do_not_autoplace no)
+			(effects
+				(font
+					(size 1.27 1.27)
+				)
+			)
+		)
+		(property "Value" "GND"
+			(at 181.61 81.2799 90)
+			(show_name no)
+			(do_not_autoplace no)
+			(effects
+				(font
+					(size 1.27 1.27)
+				)
+				(justify right)
+			)
+		)
+		(property "Footprint" ""
+			(at 177.8 81.28 0)
+			(hide yes)
+			(show_name no)
+			(do_not_autoplace no)
+			(effects
+				(font
+					(size 1.27 1.27)
+				)
+			)
+		)
+		(property "Datasheet" ""
+			(at 177.8 81.28 0)
+			(hide yes)
+			(show_name no)
+			(do_not_autoplace no)
+			(effects
+				(font
+					(size 1.27 1.27)
+				)
+			)
+		)
+		(property "Description" "Power symbol creates a global label with name \"GND\" , ground"
+			(at 177.8 81.28 0)
+			(hide yes)
+			(show_name no)
+			(do_not_autoplace no)
+			(effects
+				(font
+					(size 1.27 1.27)
+				)
+			)
+		)
+		(pin "1"
+		)
+		(instances
+			(project "Nixie Driver Tester"
+				(path "/c2082ee6-4c2e-4b3c-b2d7-410eae192cfe/394d8c35-7fb7-4f2e-9832-1fea7fce0352"
+					(reference "#PWR027")
+					(unit 1)
+				)

Commit message: switch MCU to SMT32C5
Parts:
- N1: now left out of the parts list
Changed lines of the file:
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@@
 		(body_style 1)
 		(exclude_from_sim no)
-		(in_bom yes)
+		(in_bom no)
 		(on_board yes)
 		(in_pos_files yes)
