File: Hardware/Nixie Driver ICSP Adapter/ICSP Adapter.kicad_pcb (KiCad board)
At the start: 2 copper layers, 24.1 x 33.7 mm, 5 parts

Commit message: V2 ICSP adapter
Parts:
- removed NIX1, NIX2: HDRF-2X3, Connector_PinHeader_2.54mm:PinHeader_2x03_P2.54mm_Vertical
- added L2: DAT, LED_THT:LED_D5.0mm, F.Cu at (135.9, 142.2)
- added N1: ~, Nixie:Nixie Driver V2, F.Cu at (127.0, 125.1)
- added R2: 100, Resistor_THT:R_Axial_DIN0207_L6.3mm_D2.5mm_P7.62mm_Horizontal, F.Cu at (135.9, 133.3)
- J1: renamed from ICSP0; value HDR-1X5H -> ICSP
- L1: renamed from PWR0; value LED-5MM_ROUND_GREEN -> PWR
- moved L1 33.3 mm to (120.7, 142.2), turned to 180 degrees
- moved J1 18.5 mm to (121.9, 113.7), turned to 90 degrees
- moved R1 16.0 mm to (132.1, 133.3), turned to 90 degrees
Connections:
- net LED renamed Net-(L1-K)
- J1 pad 1: ~{MCLR} -> SCLK
- J1 pad 2: VDD -> SDAT
- J1 pad 4: SDAT -> VDD
- J1 pad 5: SCLK -> ~{MCLR}
Routing:
- net GND: track 0.00 -> 24.1 mm
- net SDAT: track 10.8 -> 32.3 mm
- net SCLK: track 10.5 -> 26.8 mm
- net VDD: track 25.0 -> 38.6 mm
- net Net-(L1-K): track 5.39 -> 18.3 mm
- net Net-(L2-K): track 0.00 -> 8.89 mm
- net ~{MCLR}: track 11.5 -> 19.0 mm
- removed copper zone on B.Cu, net GND
Other:
- board size 24.1 x 33.7 mm -> 21.6 x 36.8 mm
- board text added: "Nixie Driver V2 ICSP Adapter Aaron Johnson 02/05/2025"
- board text removed: "Nixie Driver ICSP Adapter Aaron Johnson 12/13/24"

Commit message: Use symbol/footprint fields.
Parts:
- N1: value ~ -> Nixie Driver
Changed lines of the file:
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@@
 			)
 		)
-		(property "Value" "~"
+		(property "Value" "Nixie Driver"
 			(at 0 1 0)
 			(unlocked yes)
 			(layer "F.Fab")
-			(hide yes)
 			(effects
 				(font
@@
 		)
 		(property "Description" ""
+			(at 0 0 0)
+			(unlocked yes)
+			(layer "F.Fab")
+			(hide yes)
+			(effects
+				(font
+					(size 1 1)
+					(thickness 0.15)
+				)
+			)
+		)
+		(property "I2C Address" "N/A"
 			(at 0 0 0)
 			(unlocked yes)
@@
 			)
 			(layer "F.Fab")
+		)
+		(fp_text user "I2C Addr: ${I2C Address}"
+			(at 0 10.16 0)
+			(unlocked yes)
+			(layer "F.SilkS")
+			(effects
+				(font
+					(size 1 1)
+					(thickness 0.15)
+				)
+			)
 		)
 		(fp_text user "${REFERENCE}"
@@
 		)
 		(group "Board Outline"
-			(members "2db64ff1-7040-4614-9953-85404d4dfc0a" "56716110-82ed-48a7-bd64-bf89c1277af5"
-				"627c1adc-37ac-40a9-98a4-345174c5e454" "c400a9cd-19bc-4807-82e8-7779b69f4340"
-				"cf856c60-99ac-443f-be9e-06507f9d64f5" "fe0ff7db-0cbd-4dfe-b55b-997b691512ac"
+			(members "28da3a61-cebd-4f6c-9fcf-d239bab68d4a" "3aada833-eec0-4cd1-a68c-7e368148e3e4"
+				"597c2c0c-8f7f-4de6-9985-1457bdbdfd13" "7c231670-cb52-4a09-b163-09af61dd0cd5"
+				"86611d83-2856-40d4-ad4a-0cd8e4f04ed9" "b79c2f19-3b0f-4626-b352-2b6787e2b266"
 			)
 		)
@@
 		(tags "LED diameter 5.0mm 2 pins")
 		(property "Reference" "L2"
-			(at 1.27 3.81 360)
+			(at 1.27 3.81 0)
 			(layer "F.SilkS")
 			(effects
@@
 		)
 		(fp_text user "${REFERENCE}"
-			(at 1.25 0 360)
+			(at 1.25 0 0)
 			(layer "F.Fab")
 			(effects
@@
 		(tags "LED diameter 5.0mm 2 pins")
 		(property "Reference" "L1"
-			(at 1.27 3.81 360)
+			(at 1.27 3.81 0)
 			(layer "F.SilkS")
 			(effects
@@
 		)
 		(fp_text user "${REFERENCE}"
-			(at 1.25 0 360)
-			(layer "F.Fab")
-			(effects
+			(at 1.25 0 0)
+			(layer "F.Fab")
+			(effects

Commit message: Add JLC PCB silkscreen order# placeholder
Other:
- board text added: "JLCJLCJLCJLC"
Changed lines of the file:
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@@
 			(outputformat 1)
 			(mirror no)
-			(drillshape 1)
+			(drillshape 0)
 			(scaleselection 1)
-			(outputdirectory "")
+			(outputdirectory "C:/Users/aaron/Desktop/Nixie Driver ICSP Adapter Gerbers/")
 		)
 	)
@@
 		)
 	)
+	(gr_text "JLCJLCJLCJLC"
+		(at 117.221 125.857 -90)
+		(layer "F.SilkS")
+		(effects
+			(font
+				(size 1 1)
+				(thickness 0.1)
+			)
+			(justify left bottom)
+		)
+	)
